File: hardware/power_9.kicad_sch (KiCad schematic)
At the start: 20 parts, among them J11 TBC 2.54mm 10A, U8 AP63203WU, U9 XC6206P182MR

Commit message: Organize schematic
Other:
- note added: "+1V8 Regulation"
- note added: "+3V3 Regulation"
- note added: "Power I/P Connector +12V/8A"
- note added: "Sheild - GND"
- moved on the sheet: C72, C73, C74, C75, C76, C77, C78, C79, C80, C81, C82, C83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

Commit message: Link footprints to Symbols
Parts:
- C72, C73, C75, C76, C80, C81, C82, C83, C84, C85: footprint Package_TO_SOT_SMD:TSOT-23-6 -> STM32F407 Dev Kit Library:C_0805_2012Metric_Pad1.18x1.45mm_HandSolder
- C74, C77, C78, C79: footprint (none) -> STM32F407 Dev Kit Library:C_0805_2012Metric_Pad1.18x1.45mm_HandSolder
- C86: footprint Package_QFP:LQFP-48_7x7mm_P0.5mm -> STM32F407 Dev Kit Library:C_1812_4532Metric_Pad1.57x3.40mm_HandSolder
- J11: footprint (none) -> STM32F407 Dev Kit Library:TerminalBlock_Xinya_XY308-2.54-3P_1x03_P2.54mm_Horizontal
- L1: footprint (none) -> STM32F407 Dev Kit Library:L_0805_2012Metric_Pad1.05x1.20mm_HandSolder
- R26: footprint (none) -> STM32F407 Dev Kit Library:R_0805_2012Metric_Pad1.20x1.40mm_HandSolder
- U8: footprint Package_TO_SOT_SMD:TSOT-23-6 -> STM32F407 Dev Kit Library:TSOT-23-6_HandSoldering
- U9: footprint Package_TO_SOT_SMD:SOT-23-3 -> STM32F407 Dev Kit Library:SOT-23-3
Changed lines of the file:
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@@
 			)
 		)
-		(property "Footprint" "Package_TO_SOT_SMD:TSOT-23-6"
+		(property "Footprint" "STM32F407 Dev Kit Library:C_0805_2012Metric_Pad1.18x1.45mm_HandSolder"
 			(at 216.2048 129.54 0)
 			(hide yes)
@@
 			)
 		)
-		(property "Footprint" "Package_TO_SOT_SMD:TSOT-23-6"
+		(property "Footprint" "STM32F407 Dev Kit Library:C_0805_2012Metric_Pad1.18x1.45mm_HandSolder"
 			(at 68.2752 121.92 0)
 			(hide yes)
@@
 			)
 		)
-		(property "Footprint" ""
+		(property "Footprint" "STM32F407 Dev Kit Library:C_0805_2012Metric_Pad1.18x1.45mm_HandSolder"
 			(at 92.4052 74.93 0)
 			(hide yes)
@@
 			)
 		)
-		(property "Footprint" ""
+		(property "Footprint" "STM32F407 Dev Kit Library:C_0805_2012Metric_Pad1.18x1.45mm_HandSolder"
 			(at 117.8052 74.93 0)
 			(hide yes)
@@
 			)
 		)
-		(property "Footprint" "Package_QFP:LQFP-48_7x7mm_P0.5mm"
+		(property "Footprint" "STM32F407 Dev Kit Library:C_1812_4532Metric_Pad1.57x3.40mm_HandSolder"
 			(at 199.0852 72.39 0)
 			(hide yes)
@@
 			)
 		)
-		(property "Footprint" ""
+		(property "Footprint" "STM32F407 Dev Kit Library:C_0805_2012Metric_Pad1.18x1.45mm_HandSolder"
 			(at 129.2352 74.93 0)
 			(hide yes)
@@
 			)
 		)
-		(property "Footprint" "Package_TO_SOT_SMD:TSOT-23-6"
+		(property "Footprint" "STM32F407 Dev Kit Library:C_0805_2012Metric_Pad1.18x1.45mm_HandSolder"
 			(at 227.6348 129.54 0)
 			(hide yes)
@@
 			)
 		)
-		(property "Footprint" "Package_TO_SOT_SMD:TSOT-23-6"
+		(property "Footprint" "STM32F407 Dev Kit Library:C_0805_2012Metric_Pad1.18x1.45mm_HandSolder"
 			(at 115.2652 135.89 0)
 			(hide yes)
@@
 			)
 		)
-		(property "Footprint" ""
+		(property "Footprint" "STM32F407 Dev Kit Library:C_0805_2012Metric_Pad1.18x1.45mm_HandSolder"
 			(at 106.3752 74.93 0)
 			(hide yes)
@@
 			)
 		)
-		(property "Footprint" "Package_TO_SOT_SMD:TSOT-23-6"
+		(property "Footprint" "STM32F407 Dev Kit Library:C_0805_2012Metric_Pad1.18x1.45mm_HandSolder"
 			(at 126.6952 135.89 0)
 			(hide yes)
@@
 			)
 		)
-		(property "Footprint" "Package_TO_SOT_SMD:TSOT-23-6"
+		(property "Footprint" "STM32F407 Dev Kit Library:C_0805_2012Metric_Pad1.18x1.45mm_HandSolder"
 			(at 138.1252 135.89 0)
 			(hide yes)
@@
 			)
 		)
-		(property "Footprint" "Package_TO_SOT_SMD:TSOT-23-6"
+		(property "Footprint" "STM32F407 Dev Kit Library:TSOT-23-6_HandSoldering"
 			(at 99.06 147.32 0)
 			(hide yes)
@@
 			)
 		)
-		(property "Footprint" "Package_TO_SOT_SMD:TSOT-23-6"
+		(property "Footprint" "STM32F407 Dev Kit Library:C_0805_2012Metric_Pad1.18x1.45mm_HandSolder"
 			(at 177.4952 129.54 0)
 			(hide yes)
@@
 			)
 		)
-		(property "Footprint" ""
+		(property "Footprint" "STM32F407 Dev Kit Library:L_0805_2012Metric_Pad1.05x1.20mm_HandSolder"
 			(at 129.54 124.46 0)
 			(hide yes)
@@
 			)
 		)
-		(property "Footprint" ""
+		(property "Footprint" "STM32F407 Dev Kit Library:R_0805_2012Metric_Pad1.20x1.40mm_HandSolder"
 			(at 188.722 68.58 90)
 			(hide yes)
@@
 			)
 		)
-		(property "Footprint" "Package_TO_SOT_SMD:SOT-23-3"
+		(property "Footprint" "STM32F407 Dev Kit Library:SOT-23-3"
 			(at 196.85 114.935 0)
 			(hide yes)
@@
 			)
 		)
-		(property "Footprint" "Package_TO_SOT_SMD:TSOT-23-6"
+		(property "Footprint" "STM32F407 Dev Kit Library:C_0805_2012Metric_Pad1.18x1.45mm_HandSolder"
 			(at 113.9952 124.46 0)
 			(hide yes)
@@
 			)
 		)
-		(property "Footprint" "Package_TO_SOT_SMD:TSOT-23-6"
+		(property "Footprint" "STM32F407 Dev Kit Library:C_0805_2012Metric_Pad1.18x1.45mm_HandSolder"
 			(at 79.7052 121.92 0)
 			(hide yes)
@@
 			)
 		)
-		(property "Footprint" ""
+		(property "Footprint" "STM32F407 Dev Kit Library:TerminalBlock_Xinya_XY308-2.54-3P_1x03_P2.54mm_Horizontal"
 			(at 73.66 69.85 0)
 			(hide yes)
@@
 			)
 		)
-		(property "Footprint" "Package_TO_SOT_SMD:TSOT-23-6"
+		(property "Footprint" "STM32F407 Dev Kit Library:C_0805_2012Metric_Pad1.18x1.45mm_HandSolder"
 			(at 166.0652 129.54 0)
 			(hide yes)

Commit message: Convert Schematic to PCB
Parts:
- added H1, H2, H3, H4: MountingHole, STM32F407 Dev Kit Library:MountingHole_3.5mm, symbol Mechanical:MountingHole
- renumbered C75 to C73, C77 to C75, C80 to C76, C81 to C77, C83 to C79, C79 to C80, C85 to C81, C73 to C82, C86 to C83, C76 to C84, C82 to C85, C84 to C86
Other:
- note added: "Mounting Holes"
- note added: "Sheild to GND"
- note removed: "Sheild - GND"
- moved on the sheet: C83, R26

Commit message: Place components for Power section
Connections:
- net +12V: now also J11.3 (Pin_3); no longer J11.1 (Pin_1)
- net GND: now also J11.1 (Pin_1); no longer J11.3 (Pin_3)
Changed lines of the file:
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@@
 	)
 	(junction
+		(at 171.45 66.04)
+		(diameter 0)
+		(color 0 0 0 0)
+	)
+	(junction
 		(at 113.03 124.46)
 		(diameter 0)
@@
 	(wire
 		(pts
+			(xy 171.45 66.04) (xy 181.61 66.04)
+		)
+		(stroke
+			(width 0)
+			(type default)
+		)
+	)
+	(wire
+		(pts
 			(xy 78.74 113.03) (xy 88.9 113.03)
 		)
@@
 	(wire
 		(pts
-			(xy 86.36 69.85) (xy 78.74 69.85)
+			(xy 80.01 69.85) (xy 78.74 69.85)
 		)
 		(stroke
@@
 		)
 	)
-	(label "SHEILD"
-		(at 163.83 66.04 0)
+	(hierarchical_label "SHEILD"
+		(shape input)
+		(at 181.61 66.04 0)
 		(effects
 			(font
 				(size 1.27 1.27)
 			)
-			(justify left bottom)
+			(justify left)
 		)
 	)
-	(label "SHEILD"
-		(at 86.36 69.85 180)
+	(hierarchical_label "SHEILD"
+		(shape input)
+		(at 80.01 69.85 0)
 		(effects
 			(font
 				(size 1.27 1.27)
 			)
-			(justify right bottom)
+			(justify left)
 		)
 	)
@@
 	)
 	(symbol
-		(lib_id "STM32F407 Dev Kit Library:Screw_Terminal_01x03")
-		(at 73.66 69.85 0)
+		(lib_id "power:GND")
+		(at 228.6 130.81 0)
 		(mirror y)
 		(unit 1)
@@
 		(dnp no)
 		(fields_autoplaced yes)
-		(property "Reference" "J11"
-			(at 73.66 60.96 0)
+		(property "Reference" "#PWR0137"
+			(at 228.6 137.16 0)
+			(hide yes)
 			(show_name no)
 			(do_not_autoplace no)
@@
 			)
 		)
-		(property "Value" "TBC 2.54mm 10A"
-			(at 73.66 63.5 0)
+		(property "Value" "GND"
+			(at 228.6 135.89 0)
 			(show_name no)
 			(do_not_autoplace no)
@@
 			)
 		)
-		(property "Footprint" "STM32F407 Dev Kit Library:TerminalBlock_Xinya_XY308-2.54-3P_1x03_P2.54mm_Horizontal"
-			(at 73.66 69.85 0)
+		(property "Footprint" ""
+			(at 228.6 130.81 0)
 			(hide yes)
 			(show_name no)
@@
 		)
 		(property "Datasheet" ""
-			(at 73.66 69.85 0)
+			(at 228.6 130.81 0)
 			(hide yes)
 			(show_name no)
@@
 			)
 		)
-		(property "Description" "Generic screw terminal, single row, 01x03, script generated (kicad-library-utils/schlib/autogen/connector/)"
-			(at 73.66 69.85 0)
+		(property "Description" "Power symbol creates a global label with name \"GND\" , ground"
+			(at 228.6 130.81 0)
 			(hide yes)
 			(show_name no)
@@
 			)
 		)
-		(pin "2"
-		)
-		(pin "3"
-		)
 		(pin "1"
 		)
@@
 			(project "STM32F407 Dev Kit"
 				(path "/f3d27387-fbda-4c9d-aea0-93d92d34cd17/4ed455fe-d27e-4e36-92a6-b54624a52e8d"
-					(reference "J11")
+					(reference "#PWR0137")
 					(unit 1)
 				)
@@
 	)
 	(symbol
-		(lib_id "power:GND")
-		(at 228.6 130.81 0)
-		(mirror y)
+		(lib_id "STM32F407 Dev Kit Library:Screw_Terminal_01x03")
+		(at 73.66 69.85 180)
 		(unit 1)
 		(body_style 1)
@@
 		(in_pos_files yes)
 		(dnp no)
-		(fields_autoplaced yes)
-		(property "Reference" "#PWR0137"
-			(at 228.6 137.16 0)
-			(hide yes)
+		(property "Reference" "J11"
+			(at 73.66 61.722 0)
 			(show_name no)
 			(do_not_autoplace no)
@@
 			)
 		)
-		(property "Value" "GND"
-			(at 228.6 135.89 0)
+		(property "Value" "TBC 2.54mm 10A"
+			(at 73.66 64.008 0)
 			(show_name no)
 			(do_not_autoplace no)
@@
 			)
 		)
-		(property "Footprint" ""
-			(at 228.6 130.81 0)
+		(property "Footprint" "STM32F407 Dev Kit Library:TerminalBlock_Xinya_XY308-2.54-3P_1x03_P2.54mm_Horizontal"
+			(at 73.66 69.85 0)
 			(hide yes)
 			(show_name no)
@@
 		)
 		(property "Datasheet" ""
-			(at 228.6 130.81 0)
+			(at 73.66 69.85 0)
 			(hide yes)
 			(show_name no)
@@
 			)
 		)
-		(property "Description" "Power symbol creates a global label with name \"GND\" , ground"
-			(at 228.6 130.81 0)
+		(property "Description" "Generic screw terminal, single row, 01x03, script generated (kicad-library-utils/schlib/autogen/connector/)"
+			(at 73.66 69.85 0)
 			(hide yes)
 			(show_name no)
@@
 			)
 		)
+		(pin "2"
+		)
+		(pin "3"
+		)
 		(pin "1"
 		)
@@
 			(project "STM32F407 Dev Kit"
 				(path "/f3d27387-fbda-4c9d-aea0-93d92d34cd17/4ed455fe-d27e-4e36-92a6-b54624a52e8d"
-					(reference "#PWR0137")
+					(reference "J11")
 					(unit 1)
 				)

Commit message: Route Ethernet section and add global labels
Other:
- moved on the sheet: C74
Changed lines of the file:
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@@
 	)
 	(junction
-		(at 91.44 67.31)
-		(diameter 0)
-		(color 0 0 0 0)
-	)
-	(junction
 		(at 165.1 120.65)
 		(diameter 0)
@@
 	)
 	(junction
-		(at 91.44 74.93)
+		(at 92.71 74.93)
 		(diameter 0)
 		(color 0 0 0 0)
@@
 	)
 	(junction
+		(at 92.71 67.31)
+		(diameter 0)
+		(color 0 0 0 0)
+	)
+	(junction
 		(at 137.16 127)
 		(diameter 0)
@@
 	(wire
 		(pts
-			(xy 78.74 67.31) (xy 91.44 67.31)
+			(xy 78.74 67.31) (xy 92.71 67.31)
 		)
 		(stroke
@@
 	(wire
 		(pts
-			(xy 105.41 74.93) (xy 91.44 74.93)
-		)
-		(stroke
-			(width 0)
-			(type default)
-		)
-	)
-	(wire
-		(pts
 			(xy 88.9 113.03) (xy 88.9 121.92)
 		)
@@
 	(wire
 		(pts
-			(xy 91.44 74.93) (xy 78.74 74.93)
+			(xy 78.74 74.93) (xy 105.41 74.93)
 		)
 		(stroke
@@
 	(wire
 		(pts
-			(xy 91.44 67.31) (xy 128.27 67.31)
+			(xy 92.71 67.31) (xy 128.27 67.31)
 		)
 		(stroke
@@
 	(wire
 		(pts
-			(xy 91.44 66.04) (xy 91.44 67.31)
+			(xy 92.71 66.04) (xy 92.71 67.31)
 		)
 		(stroke
@@
 		)
 	)
-	(hierarchical_label "SHEILD"
+	(global_label "SHEILD"
 		(shape input)
 		(at 181.61 66.04 0)
+		(fields_autoplaced yes)
 		(effects
 			(font
@@
 			(justify left)
 		)
+		(property "Intersheetrefs" "${INTERSHEET_REFS}"
+			(at 191.1871 66.04 0)
+			(hide yes)
+			(show_name no)
+			(do_not_autoplace no)
+			(effects
+				(font
+					(size 1.27 1.27)
+				)
+				(justify left)
+			)
+		)
 	)
-	(hierarchical_label "SHEILD"
+	(global_label "SHEILD"
 		(shape input)
 		(at 80.01 69.85 0)
+		(fields_autoplaced yes)
 		(effects
 			(font
@@
 			(justify left)
 		)
+		(property "Intersheetrefs" "${INTERSHEET_REFS}"
+			(at 89.5871 69.85 0)
+			(hide yes)
+			(show_name no)
+			(do_not_autoplace no)
+			(effects
+				(font
+					(size 1.27 1.27)
+				)
+				(justify left)
+			)
+		)
 	)
 	(symbol
@@
 	(symbol
 		(lib_id "Device:C")
-		(at 91.44 71.12 0)
+		(at 92.71 71.12 0)
 		(unit 1)
 		(body_style 1)
@@
 		(fields_autoplaced yes)
 		(property "Reference" "C74"
-			(at 95.25 69.8499 0)
+			(at 96.52 69.8499 0)
 			(show_name no)
 			(do_not_autoplace no)
@@
 		)
 		(property "Value" "1000u"
-			(at 95.25 72.3899 0)
+			(at 96.52 72.3899 0)
 			(show_name no)
 			(do_not_autoplace no)
@@
 		)
 		(property "Footprint" "STM32F407 Dev Kit Library:C_0805_2012Metric_Pad1.18x1.45mm_HandSolder"
-			(at 92.4052 74.93 0)
+			(at 93.6752 74.93 0)
 			(hide yes)
 			(show_name no)
@@
 		)
 		(property "Datasheet" ""
-			(at 91.44 71.12 0)
+			(at 92.71 71.12 0)
 			(hide yes)
 			(show_name no)
@@
 		)
 		(property "Description" "Unpolarized capacitor"
-			(at 91.44 71.12 0)
+			(at 92.71 71.12 0)
 			(hide yes)
 			(show_name no)
@@
 	(symbol
 		(lib_id "power:+12V")
-		(at 91.44 66.04 0)
+		(at 92.71 66.04 0)
 		(unit 1)
 		(body_style 1)
@@
 		(fields_autoplaced yes)
 		(property "Reference" "#PWR0123"
-			(at 91.44 69.85 0)
+			(at 92.71 69.85 0)
 			(hide yes)
 			(show_name no)
@@
 		)
 		(property "Value" "+12V"
-			(at 91.44 60.96 0)
+			(at 92.71 60.96 0)
 			(show_name no)
 			(do_not_autoplace no)
@@
 		)
 		(property "Footprint" ""
-			(at 91.44 66.04 0)
+			(at 92.71 66.04 0)
 			(hide yes)
 			(show_name no)
@@
 		)
 		(property "Datasheet" ""
-			(at 91.44 66.04 0)
+			(at 92.71 66.04 0)
 			(hide yes)
 			(show_name no)
@@
 		)
 		(property "Description" "Power symbol creates a global label with name \"+12V\""
-			(at 91.44 66.04 0)
+			(at 92.71 66.04 0)
 			(hide yes)
 			(show_name no)

Commit message: Fix capacitor footprints
Parts:
- C74: footprint STM32F407 Dev Kit Library:C_0805_2012Metric_Pad1.18x1.45mm_HandSolder -> STM32F407 Dev Kit Library:CP_Elec_10x12.5
- C75: footprint STM32F407 Dev Kit Library:C_0805_2012Metric_Pad1.18x1.45mm_HandSolder -> STM32F407 Dev Kit Library:C_1210_3225Metric_Pad1.33x2.70mm_HandSolder
Changed lines of the file:
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@@
 			)
 		)
-		(property "Footprint" "STM32F407 Dev Kit Library:C_0805_2012Metric_Pad1.18x1.45mm_HandSolder"
+		(property "Footprint" "STM32F407 Dev Kit Library:CP_Elec_10x12.5"
 			(at 93.6752 74.93 0)
 			(hide yes)
@@
 			)
 		)
-		(property "Footprint" "STM32F407 Dev Kit Library:C_0805_2012Metric_Pad1.18x1.45mm_HandSolder"
+		(property "Footprint" "STM32F407 Dev Kit Library:C_1210_3225Metric_Pad1.33x2.70mm_HandSolder"
 			(at 106.3752 74.93 0)
 			(hide yes)

Commit message: Add prices to BOM
Parts:
- R26: value 1M -> 1M 2kV
Other:
- moved on the sheet: R26
Changed lines of the file:
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@@
 	(wire
 		(pts
-			(xy 163.83 74.93) (xy 163.83 73.66)
+			(xy 158.75 74.93) (xy 158.75 73.66)
 		)
 		(stroke
@@
 	(wire
 		(pts
-			(xy 163.83 66.04) (xy 171.45 66.04)
+			(xy 158.75 66.04) (xy 171.45 66.04)
 		)
 		(stroke
@@
 	(symbol
 		(lib_id "STM32F407 Dev Kit Library:R")
-		(at 163.83 69.85 0)
+		(at 158.75 69.85 0)
 		(unit 1)
 		(body_style 1)
@@
 		(dnp no)
 		(property "Reference" "R26"
-			(at 165.354 68.58 0)
+			(at 160.274 68.58 0)
 			(show_name no)
 			(do_not_autoplace no)
@@
 			)
 		)
-		(property "Value" "1M"
-			(at 165.354 71.12 0)
+		(property "Value" "1M 2kV"
+			(at 160.274 71.12 0)
 			(show_name no)
 			(do_not_autoplace no)
@@
 		)
 		(property "Footprint" "STM32F407 Dev Kit Library:R_0805_2012Metric_Pad1.20x1.40mm_HandSolder"
-			(at 162.052 69.85 90)
+			(at 156.972 69.85 90)
 			(hide yes)
 			(show_name no)
@@
 		)
 		(property "Datasheet" ""
-			(at 163.83 69.85 0)
+			(at 158.75 69.85 0)
 			(hide yes)
 			(show_name no)
@@
 		)
 		(property "Description" "Resistor"
-			(at 163.83 69.85 0)
+			(at 158.75 69.85 0)
 			(hide yes)
 			(show_name no)
@@
 	(symbol
 		(lib_id "power:GND")
-		(at 163.83 74.93 0)
+		(at 158.75 74.93 0)
 		(unit 1)
 		(body_style 1)
@@
 		(fields_autoplaced yes)
 		(property "Reference" "#PWR0129"
-			(at 163.83 81.28 0)
+			(at 158.75 81.28 0)
 			(hide yes)
 			(show_name no)
@@
 		)
 		(property "Value" "GND"
-			(at 163.83 80.01 0)
+			(at 158.75 80.01 0)
 			(show_name no)
 			(do_not_autoplace no)
@@
 		)
 		(property "Footprint" ""
-			(at 163.83 74.93 0)
+			(at 158.75 74.93 0)
 			(hide yes)
 			(show_name no)
@@
 		)
 		(property "Datasheet" ""
-			(at 163.83 74.93 0)
+			(at 158.75 74.93 0)
 			(hide yes)
 			(show_name no)
@@
 		)
 		(property "Description" "Power symbol creates a global label with name \"GND\" , ground"
-			(at 163.83 74.93 0)
+			(at 158.75 74.93 0)
 			(hide yes)
 			(show_name no)
